File: ESP32 Robo Dev Board/Range Finder Array.kicad_sch (KiCad schematic)
At the start: 24 parts

Commit message: First Finished Version 0.1.
Parts:
- renumbered R408 to R10, R409 to R11, R410 to R12, R411 to R13, R412 to R14, R413 to R15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
