File: Hardware/Range Finder Array.kicad_sch (KiCad schematic)
At the start: 32 parts, among them U10 VL53L1CXV0FY1, U11 VL53L1CXV0FY1, U12 VL53L1CXV0FY1, U13 VL53L1CXV0FY1, U6 VL53L1CXV0FY1, U7 VL53L1CXV0FY1, U9 VL53L1CXV0FY1

Commit message: BIG Changes
Create a 4 Layer Variation
Change Motor Controller routing.
Change Power Regulation.
Optimize Sensor routing.
Pray I know what i'm doing
Parts:
- C10, C11, C13, C14, C15, C16, C17, C18, C19, C20, C21, C22, C7, C8: footprint Capacitor_SMD:C_0805_2012Metric -> Capacitor_SMD:C_0603_1608Metric
- C12: value (none) -> 4.7 uF; footprint (none) -> Capacitor_SMD:C_0603_1608Metric
- C9: value (none) -> 100 nF; footprint (none) -> Capacitor_SMD:C_0603_1608Metric
- R3: footprint Resistor_SMD:R_0805_2012Metric -> Resistor_SMD:R_0603_1608Metric
- R5: value (none) -> 10K; footprint (none) -> Resistor_SMD:R_0805_2012Metric
- U8: value (none) -> VL53L1CXV0FY1; footprint (none) -> Sensor_Distance:ST_VL53L1x

Commit message: 4 L:ayer Board with USB-C
Created a 4-Layer PCB with USB-C updates
Parts:
- removed C10, C11, C12, C16, C17, C18, C21, C22: 4.7 uF, Capacitor_SMD:C_0603_1608Metric, symbol Device:C_Small
- removed C13, C14, C15, C19, C20, C7, C8, C9: 100 nF, Capacitor_SMD:C_0603_1608Metric, symbol Device:C_Small
- removed R10, R4, R5, R6, R7, R8, R9: 10K, Resistor_SMD:R_0805_2012Metric, symbol Device:R_Small
- removed R3: 10K, Resistor_SMD:R_0603_1608Metric, symbol Device:R_Small
- removed U10, U11, U12, U13, U6, U7, U8, U9: VL53L1CXV0FY1, Sensor_Distance:ST_VL53L1x, symbol Sensor_Distance:VL53L1CXV0FY1
Connections:
- no-connect marks 8 -> 0
