File: Hardware/USB C Interface.kicad_sch (KiCad schematic)
At the start: 5 parts, among them J1 USB_C_Receptacle_USB2.0, U6 USBLC6-2P6

Commit message: Clean Up Schematic
Fixed Schematic notes, and formatting
Other:
- title: (none) -> USB C Connector
Changed lines of the file:
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@@
 	(generator_version "9.0")
 	(paper "A4")
+	(title_block
+		(title "USB C Connector")
+	)
 	(text "This implementation of USB-C should allow for the user to utilize \nUSB2.0 Speed data connection. Furthermore, the end-user will be able \nto charge the battery pack, program the ESP32, and use it for serial \ndebugging."
 		(exclude_from_sim no)
